File: Kosmodulator.kicad_sch (KiCad schematic)
At the start: 6 parts

Commit message: schem complete
Parts:
- added C1, C2: 100n, symbol Device:C_Small
- added C3: C, symbol Device:C
- added D1, D2: D, symbol Device:D
- added J1, J2, J3, J4, J5: AudioJack2, symbol Connector:AudioJack2
- added J6: Conn_02x05_Odd_Even, symbol Connector_Generic:Conn_02x05_Odd_Even
- added R1, R10, R11, R8, R9: 100K, symbol Device:R
- added R12, R13, R14, R15: 1K, symbol Device:R
- added R2, R3, R4, R5, R6, R7: R, symbol Device:R
- added RV2, RV3, RV4, RV5: 100K, symbol Device:R_POT_TRIM
- added SW1, SW2, SW3: SW_Rotary12, symbol Switch:SW_Rotary12
- gave numbers to parts that had none: 2
Connections:
- net at U1.12 (+): now also C3.2, SW3.13
- net at U1.13 (-): now also U1.14, R14.1, R8.1
- net at RV1.1: now also SW1.13
- net at RV1.2: now also U1.5 (+), C3.1
- net at RV1.3: now also SW2.13
- net at U1.6 (-): now also U1.7, R15.1, R9.1
- net GND: now reaches U1.10 (+)
- net GND: now also U1.3 (+), C1.2, C2.2, J1.S, J2.S, J3.S, J4.S, J5.S, J6.3 (Pin_3), J6.4 (Pin_4), J6.5 (Pin_5), J6.6 (Pin_6), J6.7 (Pin_7), J6.8 (Pin_8), R2.2, R3.2, R4.2, R5.2, R6.2, R7.2, RV2.1, RV3.1, RV4.1, RV5.1, SW1.1, SW2.4
- net at U1.8: now also R11.2, R12.1
- net at U1.9 (-): now also R11.1, R8.2
- net at U1.1: now also R10.2, R13.1
- net at U1.2 (-): now also R10.1, R9.2
- net -12V: now reaches U1.11 (V-)
- net -12V: now also C1.1, D2.2 (A), RV2.3, RV3.3
- net +12V: now reaches U1.4 (V+)
- net +12V: now also C2.1, D1.1 (K), RV4.3, RV5.3
- new net: J4.T, R13.2
- new net: J3.T, R14.2
- new net: R6.1, SW3.2
- new net: R7.1, SW3.1
- new net: R5.1, SW3.3
- new net: R4.1, SW3.4
- new net: R3.1, SW3.5
- new net: R2.1, SW3.6
- new net: J1.T, R1.1
- new net: R1.2, SW2.1
- new net: RV2.2, SW1.3
- new net: D2.1 (K), J6.1 (Pin_1), J6.2 (Pin_2)
- new net: D1.2 (A), J6.10 (Pin_10), J6.9 (Pin_9)
- new net: RV3.2, SW1.2
- new net: RV5.2, SW2.2
- new net: J2.T, R12.2
- new net: J5.T, R15.2
- new net: RV4.2, SW2.3
- no-connect marks 0 -> 23
Other:
- moved on the sheet: U1A, U1B, U1C, U1D
